File: Monitor/Monitor.kicad_pcb (KiCad board)
At the start: 2 copper layers, 11 parts, among them U1 ESP32-S3-WROOM-1, U10 SSD1306, U11 USBLC6-2SC6, U2 AMS1117-3.3, U3 AP2112K-3.0, U4 TMP102xxDRL, U5 LTR-303ALS-01, U6 AHT20, U7 AGS10, U8 BMP388, U9 BQ24075RGT

Commit message: Finish PCB + pictures + BOM
Parts:
- added C1: 100n, Capacitor_SMD:C_0603_1608Metric, F.Cu at (144.4, 76.8)
- added C10: 4u7, Capacitor_SMD:C_0603_1608Metric, F.Cu at (147.4, 80.1)
- added C11: 4u7, Capacitor_SMD:C_0603_1608Metric, F.Cu at (150.3, 94.9)
- added C12: 100n, Capacitor_SMD:C_0603_1608Metric, F.Cu at (137.0, 61.6)
- added C13: 100n, Capacitor_SMD:C_0603_1608Metric, F.Cu at (110.1, 85.5)
- added C14: 100n, Capacitor_SMD:C_0603_1608Metric, F.Cu at (149.1, 72.2)
- added C15: 100n, Capacitor_SMD:C_0603_1608Metric, F.Cu at (117.6, 98.7)
- added C16: 100n, Capacitor_SMD:C_0603_1608Metric, F.Cu at (110.1, 82.8)
- added C17: 100n, Capacitor_SMD:C_0603_1608Metric, F.Cu at (144.5, 64.5)
- added C18: 100n, Capacitor_SMD:C_0603_1608Metric, F.Cu at (147.3, 97.9)
- added C2: 4u7, Capacitor_SMD:C_0603_1608Metric, F.Cu at (129.7, 83.4)
- added C3: 4u7, Capacitor_SMD:C_0603_1608Metric, F.Cu at (134.2, 81.3)
- added C4: 100n, Capacitor_SMD:C_0603_1608Metric, F.Cu at (123.3, 89.7)
- added C5: 4u7, Capacitor_SMD:C_0603_1608Metric, F.Cu at (138.8, 86.1)
- added C6: 4u7, Capacitor_SMD:C_0603_1608Metric, F.Cu at (136.4, 90.0)
- added C7: 100n, Capacitor_SMD:C_0603_1608Metric, F.Cu at (133.1, 71.5)
- added C8: 4u7, Capacitor_SMD:C_0603_1608Metric, F.Cu at (142.7, 94.8)
- added C9: 4u7, Capacitor_SMD:C_0603_1608Metric, F.Cu at (141.6, 83.7)
- added D1: PGD, LED_SMD:LED_1206_3216Metric, F.Cu at (115.1, 85.8)
- added D2: CHG, LED_SMD:LED_1206_3216Metric, F.Cu at (120.7, 85.8)
- added J1: USB_C_Receptacle_USB2.0_14P, Connector_USB:USB_C_Receptacle_G-Switch_GT-USB-7010ASV, F.Cu at (125.0, 96.0)
- added J2: BAT, Connector_JST:JST_PH_B2B-PH-K_1x02_P2.00mm_Vertical, F.Cu at (135.7, 95.2)
- added R1: 3k, Resistor_SMD:R_0603_1608Metric, F.Cu at (131.8, 81.3)
- added R10: 10k, Resistor_SMD:R_0603_1608Metric, F.Cu at (117.6, 89.0)
- added R11: 10k, Resistor_SMD:R_0603_1608Metric, F.Cu at (120.2, 89.0)
- added R12: 2k2, Resistor_SMD:R_0603_1608Metric, F.Cu at (130.2, 76.9)
- added R13: 2k2, Resistor_SMD:R_0603_1608Metric, F.Cu at (130.2, 73.6)
- added R14: 5k1, Resistor_SMD:R_0603_1608Metric, F.Cu at (148.8, 64.4)
- added R2: 62k, Resistor_SMD:R_0603_1608Metric, F.Cu at (129.7, 86.3)
- added R3: 4k3, Resistor_SMD:R_0603_1608Metric, F.Cu at (129.7, 88.6)
- added R4: 5k1, Resistor_SMD:R_0603_1608Metric, F.Cu at (117.6, 92.4)
- added R5: 5k1, Resistor_SMD:R_0603_1608Metric, F.Cu at (117.6, 95.9)
- added R6: 10k, Resistor_SMD:R_0603_1608Metric, F.Cu at (132.4, 91.5)
- added R7: 1k, Resistor_SMD:R_0603_1608Metric, F.Cu at (114.5, 82.9)
- added R8: 1k, Resistor_SMD:R_0603_1608Metric, F.Cu at (119.8, 82.9)
- added R9: 5k1, Resistor_SMD:R_0603_1608Metric, F.Cu at (138.5, 64.5)
- added SW1: RST, Button_Switch_SMD:SW_SPST_PTS647_Sx38, F.Cu at (111.9, 90.4)
- added SW2: BOOT, Button_Switch_SMD:SW_SPST_PTS647_Sx38, F.Cu at (111.9, 96.8)
- U1: value ESP32-S3-WROOM-1 -> AGS10; footprint RF_Module:ESP32-S3-WROOM-1 -> AGS10:AGS10
- U10: value SSD1306 -> ESP32-S3-WROOM-1; footprint Display:ER_OLEDM0.91_1x-I2C -> RF_Module:ESP32-S3-WROOM-1
- U11: value USBLC6-2SC6 -> SSD1306; footprint Package_TO_SOT_SMD:SOT-23-6 -> Display:ER_OLEDM0.91_1x-I2C
- U2: value AMS1117-3.3 -> BQ24075RGT; footprint Package_TO_SOT_SMD:SOT-223-3_TabPin2 -> Package_DFN_QFN:VQFN-16-1EP_3x3mm_P0.5mm_EP1.6x1.6mm
- U3: value AP2112K-3.0 -> USBLC6-2SC6; footprint Package_TO_SOT_SMD:SOT-23-5 -> Package_TO_SOT_SMD:SOT-23-6
- U4: value TMP102xxDRL -> BMP388; footprint Package_TO_SOT_SMD:SOT-563 -> BMP388:XDCR_BMP388
- U5: value LTR-303ALS-01 -> AMS1117-3.3; footprint OptoDevice:Lite-On_LTR-303ALS-01 -> Package_TO_SOT_SMD:SOT-223-3_TabPin2
- U6: value AHT20 -> AP2112K-3.0; footprint AHT20:PSON100P300X300X110-6N -> Package_TO_SOT_SMD:SOT-23-5
- U7: value AGS10 -> LTR-303ALS-01; footprint AGS10:AGS10 -> OptoDevice:Lite-On_LTR-303ALS-01
- U8: value BMP388 -> AHT20; footprint BMP388:XDCR_BMP388 -> AHT20:PSON100P300X300X110-6N
- U9: value BQ24075RGT -> TMP102xxDRL; footprint Package_DFN_QFN:VQFN-16-1EP_3x3mm_P0.5mm_EP1.6x1.6mm -> Package_TO_SOT_SMD:SOT-563
- moved U10 82.9 mm to (114.8, 71.3), turned to 90 degrees
- moved U3 71.1 mm to (125.5, 86.1), turned to 90 degrees
- moved U4 48.4 mm to (137.0, 71.8), turned to 90 degrees
- moved U7 41.0 mm to (136.0, 64.5), turned to -90 degrees
- moved U9 37.9 mm to (146.7, 64.5), turned to 90 degrees
- moved U8 34.7 mm to (146.0, 72.0), turned to 90 degrees
- moved U11 32.5 mm to (163.5, 97.5), turned to 180 degrees
- moved U5 31.1 mm to (146.6, 86.0), turned to -90 degrees
- moved U6 27.6 mm to (146.5, 95.0)
- moved U1 27.3 mm to (141.7, 78.8), turned to -90 degrees
- moved U2 20.7 mm to (134.2, 85.9), turned to 90 degrees
Connections:
- U1 pad 1: GND -> /SCL
- U1 pad 2: +3V3 -> /SDA
- U1 pad 3: Net-(U1-EN) -> GND
- U1 pad 4: unconnected-(U1-IO4-Pad4) -> +3V0
- U10 pad 2: unconnected-(U10-VCC-Pad2) -> +3V3
- U10 pad 3: unconnected-(U10-SCL-Pad3) -> Net-(U10-EN)
- U11 pad 1: /D- -> GND
- U11 pad 2: GND -> +3V3
- U11 pad 3: /D+ -> /SCL
- U11 pad 4: /D+OUT -> /SDA
- U2 pad 1: GND -> Net-(U2-TS)
- U2 pad 2: +3V3 -> /BAT+
- U2 pad 3: +5V -> /BAT+
- U3 pad 1: +5V -> /D-
- U3 pad 3: +5V -> /D+
- U3 pad 4: unconnected-(U3-NC-Pad4) -> /DOut+
- U3 pad 5: +3V0 -> +5V
- U4 pad 1: unconnected-(U4-SCL-Pad1) -> +3V3
- U4 pad 2: GND -> /SCK
- U4 pad 3: unconnected-(U4-ALERT-Pad3) -> GND
- U4 pad 4: unconnected-(U4-ADD0-Pad4) -> /MOSI
- U4 pad 5: unconnected-(U4-V+-Pad5) -> /MISO
- U4 pad 6: unconnected-(U4-SDA-Pad6) -> /CSB
- U5 pad 1: unconnected-(U5-VDD-Pad1) -> GND
- U5 pad 2: unconnected-(U5-NC-Pad2) -> +3V3
- U5 pad 3: GND -> VCC
- U6 pad 1: unconnected-(U6-NC-Pad1) -> VCC
- U6 pad 2: unconnected-(U6-VDD-Pad2) -> GND
- U6 pad 3: unconnected-(U6-SCL-Pad3) -> VCC
- U6 pad 5: GND -> +3V0
- U7 pad 1: unconnected-(U7-SCL-Pad1) -> +3V3
- U7 pad 4: unconnected-(U7-VCC-Pad4) -> /SCL
- U8 pad 2: unconnected-(U8-SCK-Pad2) -> +3V3
- U8 pad 3: GND -> /SCL
- U8 pad 4: unconnected-(U8-SDI-Pad4) -> /SDA
- U8 pad 5: unconnected-(U8-SDO-Pad5) -> GND
- U9 pad 1: unconnected-(U9-TS-Pad1) -> /SCL
- U9 pad 2: Net-(U9-BAT-Pad2) -> GND
- U9 pad 3: Net-(U9-BAT-Pad2) -> /ALRT
- U9 pad 4: unconnected-(U9-~{CE}-Pad4) -> GND
- U9 pad 5: unconnected-(U9-EN2-Pad5) -> +3V3
- U9 pad 6: unconnected-(U9-EN1-Pad6) -> /SDA
Routing:
- net +3V3: track 0.00 -> 151.3 mm, vias 0 -> 5
- net /SDA: track 0.00 -> 85.8 mm, vias 0 -> 5
- net /SCL: track 0.00 -> 82.5 mm, vias 0 -> 5
- net Net-(U10-IO0): track 0.00 -> 51.3 mm, vias 0 -> 4
- net VCC: track 0.00 -> 35.1 mm
- net /ALRT: track 0.00 -> 35.1 mm
- net +5V: track 0.00 -> 31.0 mm
- net +3V0: track 0.00 -> 27.9 mm, vias 0 -> 2
- net /INT: track 0.00 -> 26.8 mm
- net Net-(D1-K): track 0.00 -> 26.4 mm, vias 0 -> 2
- net Net-(D2-K): track 0.00 -> 21.1 mm, vias 0 -> 2
- net Net-(U10-EN): track 0.00 -> 19.8 mm, vias 0 -> 2
- net /MOSI: track 0.00 -> 13.8 mm
- net /MISO: track 0.00 -> 11.8 mm
- net Net-(J1-CC2): track 0.00 -> 11.6 mm, vias 0 -> 2
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- added copper zone on B.Cu, net GND
- added copper zone on F.Cu, net GND
- added copper zone on F.Cu, net VCC
Other:
- board outline added: 59.5 x 40 mm
- rule pad_to_mask_clearance: 0 -> 0.05
- board text added: "DYNIX"
